Commit message: gazebo対応

File: patches/turtlebot_common_library.urdf.xacro (robot description, xacro)
@@ -7,5 +7,6 @@
   <xacro:include filename="$(find turtlebot_description)/urdf/common_properties.urdf.xacro"/>
   <xacro:include filename="$(find turtlebot_description)/urdf/turtlebot_properties.urdf.xacro"/>
-  <joint name="laser_frame" type="fixed">
+  <!--実機用-->
+  <joint name="laser_joint" type="fixed">
     <origin xyz="0.1 0.0 0.3" rpy="0 0 3.14" />
     <parent link="base_link" />
@@ -27,3 +28,22 @@
     </inertial>
   </link>
+  <!--Gazebo用-->
+  <!--Gazeboではgeometryのboxがあると何故かエラーを吐くため-->
+  <!--joint name="laser_frame" type="fixed">
+    <origin xyz="0.1 0.0 0.35" rpy="0 0 0" />
+    <parent link="base_link" />
+    <child link="laser_frame" />
+  </joint>
+  <link name="laser_frame">
+    <visual>
+      <material name="Green" />
+    </visual>
+    <inertial>
+      <mass value="0.000001" />
+      <origin xyz="0 0 0" />
+      <inertia ixx="0.0001" ixy="0.0" ixz="0.0"
+        iyy="0.0001" iyz="0.0"
+        izz="0.0001" />
+    </inertial>
+  </link-->
 </robot>

File: patches/turtlebot_gazebo.urdf.xacro (robot description, xacro)
@@ -38,9 +38,7 @@
         </plugin>
       </sensor>
-    </gazebo>
- <!-- hokuyo -->
-  <gazebo reference="hokuyo_link">
-    <sensor type="gpu_ray" name="head_hokuyo_sensor">
-      <pose>0 0 0 0 0 0</pose>
+      <!--GazebooのLidar-->
+      <sensor type="gpu_ray" name="head_hokuyo_sensor">
+      <pose>1 1 1 0 0 0</pose>
       <visualize>false</visualize>
       <update_rate>40</update_rate>
@@ -50,19 +48,15 @@
             <samples>720</samples>
             <resolution>1</resolution>
-            <min_angle>-1.570796</min_angle>
-            <max_angle>1.570796</max_angle>
+            <min_angle>-3.141592</min_angle>
+            <max_angle>3.141592</max_angle>
           </horizontal>
         </scan>
         <range>
           <min>0.10</min>
-          <max>30.0</max>
+          <max>10.0</max>
           <resolution>0.01</resolution>
         </range>
         <noise>
           <type>gaussian</type>
-          <!-- Noise parameters based on published spec for Hokuyo laser
-               achieving "+-30mm" accuracy at range < 10m.  A mean of 0.0m and
-               stddev of 0.01m will put 99.7% of samples within 0.03m of the true
-               reading. -->
           <mean>0.0</mean>
           <stddev>0.01</stddev>
@@ -70,9 +64,9 @@
       </ray>
       <plugin name="gazebo_ros_head_hokuyo_controller" filename="libgazebo_ros_gpu_laser.so">
-        <topicName>/rrbot/laser/scan</topicName>
-        <frameName>hokuyo_link</frameName>
+        <topicName>/scan</topicName>
+        <frameName>laser_frame</frameName>
       </plugin>
     </sensor>
-  </gazebo>
+    </gazebo>
   </xacro:macro>
 </robot>

Commit message: lidar修正

File: patches/turtlebot_common_library.urdf.xacro (robot description, xacro)
@@ -9,5 +9,5 @@
   <!--実機用-->
   <joint name="laser_joint" type="fixed">
-    <origin xyz="0.1 0.0 0.3" rpy="0 0 3.14" />
+    <origin xyz="0.1 0.0 0.3" rpy="0 0 0" />
     <parent link="base_link" />
     <child link="laser_frame" />

Commit message: Update turtlebot_common_library.urdf.xacro

File: patches/turtlebot_common_library.urdf.xacro (robot description, xacro)
@@ -7,7 +7,6 @@
   <xacro:include filename="$(find turtlebot_description)/urdf/common_properties.urdf.xacro"/>
   <xacro:include filename="$(find turtlebot_description)/urdf/turtlebot_properties.urdf.xacro"/>
-  <!--実機用-->
-  <joint name="laser_joint" type="fixed">
-    <origin xyz="0.1 0.0 0.3" rpy="0 0 3.14" />
+  <joint name="laser_frame" type="fixed">
+    <origin xyz="0.1 0.0 0.35" rpy="0 0 0" />
     <parent link="base_link" />
     <child link="laser_frame" />
@@ -15,7 +14,7 @@
   <link name="laser_frame">
     <visual>
-      <geometry>
+      <!--geometry>
         <box size="0.00 0.05 0.06" />
-      </geometry>
+      </geometry-->
       <material name="Green" />
     </visual>
@@ -28,22 +27,3 @@
     </inertial>
   </link>
-  <!--Gazebo用-->
-  <!--Gazeboではgeometryのboxがあると何故かエラーを吐くため-->
-  <!--joint name="laser_frame" type="fixed">
-    <origin xyz="0.1 0.0 0.35" rpy="0 0 0" />
-    <parent link="base_link" />
-    <child link="laser_frame" />
-  </joint>
-  <link name="laser_frame">
-    <visual>
-      <material name="Green" />
-    </visual>
-    <inertial>
-      <mass value="0.000001" />
-      <origin xyz="0 0 0" />
-      <inertia ixx="0.0001" ixy="0.0" ixz="0.0"
-        iyy="0.0001" iyz="0.0"
-        izz="0.0001" />
-    </inertial>
-  </link-->
 </robot>

Commit message: [fix] バグっていた文字列部分を消去

File: patches/turtlebot_common_library.urdf.xacro (robot description, xacro)
@@ -7,12 +7,6 @@
   <xacro:include filename="$(find turtlebot_description)/urdf/common_properties.urdf.xacro"/>
   <xacro:include filename="$(find turtlebot_description)/urdf/turtlebot_properties.urdf.xacro"/>
-<<<<<<< HEAD
-  <!--Robot-->
-  <joint name="laser_joint" type="fixed">
-    <origin xyz="0.1 0.0 0.3" rpy="0 0 0" />
-=======
   <joint name="laser_frame" type="fixed">
     <origin xyz="0.1 0.0 0.35" rpy="0 0 0" />
->>>>>>> ad6968fa2cd8b14cad4e7873de04748f032cbe5f
     <parent link="base_link" />
     <child link="laser_frame" />
@@ -20,7 +14,7 @@
   <link name="laser_frame">
     <visual>
-      <!--geometry>
+      <geometry>
         <box size="0.00 0.05 0.06" />
-      </geometry-->
+      </geometry>
       <material name="Green" />
     </visual>
@@ -33,5 +27,4 @@
     </inertial>
   </link>
-<<<<<<< HEAD
   <!--Gazebo-->
   <!--joint name="laser_frame" type="fixed">
@@ -52,5 +45,3 @@
     </inertial>
   </link-->
-=======
->>>>>>> ad6968fa2cd8b14cad4e7873de04748f032cbe5f
 </robot>
